Commit message: add gazebo agilex

File: SemanticMap/octomap_generator_ws/src/agilex_description/urdf/xacro/gazebo/agilex_mini_gazebo.xacro (robot description, xacro)
@@ -1,10 +1,7 @@
 <?xml version="1.0"?>
-<robot xmlns:xacro="http://www.ros.org/wiki/xacro"
-    xmlns:sensor="http://playerstage.sourceforge.net/gazebo/xmlschema/#sensor"
-    xmlns:controller="http://playerstage.sourceforge.net/gazebo/xmlschema/#controller"
-    xmlns:interface="http://playerstage.sourceforge.net/gazebo/xmlschema/#interface" name="robot">
+<robot name="agilex_mini"
+    xmlns:xacro="http://www.ros.org/wiki/xacro">
     <xacro:property name="length_wheel" value="0.05" />
     <xacro:property name="radius_wheel" value="0.05" />
-    <xacro:property name="camera_link" value="0.05" />
     <xacro:macro name="default_inertial" params="mass">
         <inertial>
@@ -22,9 +19,9 @@
         <xacro:default_inertial mass="0.0001"/>
     </link>
-    <xacro:include filename="$(find agilex_description)/urdf/xacro/gazebo/robot.gazebo" />
     <gazebo reference="base_footprint">
         <material>Gazebo/Green</material>
         <turnGravityOff>false</turnGravityOff>
     </gazebo>
+    <xacro:include filename="$(find agilex_description)/urdf/xacro/gazebo/agilex_mini_gazebo.gazebo" />
     <joint name="base_footprint_joint" type="fixed">
         <origin xyz="0 0 0" />
@@ -141,25 +138,24 @@
         <origin rpy="-1.5707 0 0" xyz="-0.1 -0.15 0"/>
     </joint>
-    <!-- Camera joint -->
-    <joint name="camera_joint" type="fixed">
-        <axis xyz="0 1 0" />
-        <origin xyz="0.125 0 0.125" rpy="0 0 0"/>
-        <parent link="base_link"/>
-        <child link="camera_link"/>
-    </joint>
-    <!-- Camera -->
-    <link name="camera_link">
-        <collision>
-            <origin xyz="0 0 0" rpy="0 0 0"/>
-            <geometry>
-                <box size="0.05 0.05 0.05"/>
-            </geometry>
-        </collision>
-        <visual>
-            <origin xyz="0 0 0" rpy="0 0 1.5707"/>
-            <geometry>
-                 <!-- <box size="0.05 0.05 0.05"/> -->
-                 <mesh filename="package://agilex_description/meshes/kinect.dae" />
-                 <!-- <mesh filename="http://models.gazebosim.org/kinect/meshes/kinect.dae" /> -->
+    <link name="sensor_support">
+        <visual>
+            <geometry>
+                <box size=".06 .16 .10"/>
+            </geometry>
+            <material name="white">
+                <color rgba="1 1 1 1"/>
+            </material>
+        </visual>
+    </link>
+    <joint name="sensor_support_joint" type="fixed">
+        <parent link="base_link"/>
+        <child link="sensor_support"/>
+        <origin rpy="0 0 0" xyz="0.10 0 0.15"/>
+    </joint>
+    <link name="zed_camera">
+        <visual>
+            <origin xyz="0 0 0" rpy="0 0 0"/>
+            <geometry>
+                <box size=".03 .14 .03"/>
             </geometry>
             <material name="red">
@@ -172,27 +168,32 @@
             <inertia ixx="1e-6" ixy="0" ixz="0" iyy="1e-6" iyz="0" izz="1e-6" />
         </inertial>
-    </link>
-    <!-- Hokuyo joint -->
-    <joint name="hokuyo_joint" type="fixed">
-        <origin xyz="0.125 0.05 0.125" rpy="0 0 0"/>
-        <parent link="base_link"/>
+        <collision>
+            <origin xyz="0 0 0" rpy="0 0 0"/>
+            <geometry>
+                <box size="0.05 0.05 0.05"/>
+            </geometry>
+        </collision>
+    </link>
+    <joint name="zed_joint" type="fixed">
         <axis xyz="0 1 0" />
-        <child link="hokuyo_link"/>
-    </joint>
-    <!-- Hokuyo Laser -->
-    <link name="hokuyo_link">
-        <collision>
-            <origin xyz="0 0 0" rpy="0 0 0"/>
-            <geometry>
-                <box size="0.1 0.1 0.1"/>
-            </geometry>
-        </collision>
-        <visual>
-            <origin xyz="0 0 0" rpy="0 0 0"/>
-            <geometry>
-                <!-- <mesh filename="http://models.gazebosim.org/hokuyo/meshes/hokuyo.dae"/> -->
-                <box size="0.1 0.1 0.1"/>
-            </geometry>
-        </visual>
+        <origin xyz="0.045 0 0.02" rpy="0 0 0"/>
+        <parent link="sensor_support"/>
+        <child link="zed_camera"/>
+    </joint>
+    <link name="rslidar">
+        <visual>
+            <geometry>
+                <cylinder length = "0.03" radius = "0.03"/>
+            </geometry>
+            <material name="white">
+                <color rgba="1 1 1 1"/>
+            </material>
+        </visual>
+        <collision>
+            <origin xyz="0 0 0" rpy="0 0 0"/>
+            <geometry>
+                <cylinder length = "0.03" radius = "0.03"/>
+            </geometry>
+        </collision>
         <inertial>
             <mass value="1e-5" />
@@ -201,3 +202,9 @@
         </inertial>
     </link>
+    <joint name="rslidar_joint" type="fixed">
+        <axis xyz="0 1 0" />
+        <origin xyz="0 0 0.065" rpy="0 0 0"/>
+        <parent link="sensor_support"/>
+        <child link="rslidar"/>
+    </joint>
 </robot>

File: SemanticMap/octomap_generator_ws/src/agilex_description/urdf/xacro/gazebo/agilex_scout_base_gazebo.xacro (robot description, xacro)
@@ -5,10 +5,18 @@
     <xacro:property name="base_mass"   value="20" />
     <xacro:property name="base_radius" value="0.20"/>
-    <xacro:property name="base_length" value="0.16"/>
+    <xacro:property name="base_length" value="0.207"/>
+    <xacro:property name="base_x" value="0.93"/>
+    <xacro:property name="base_y" value="0.467"/>
+    <xacro:property name="base_z" value="0.207"/>
+    <xacro:property name="base_box_x" value="0.738"/>
+    <xacro:property name="base_box_y" value="0.248"/>
+    <xacro:property name="base_box_z" value="0.17"/>
     <xacro:property name="wheel_mass"   value="2" />
-    <xacro:property name="wheel_radius" value="0.06"/>
-    <xacro:property name="wheel_length" value="0.025"/>
-    <xacro:property name="wheel_joint_y" value="0.19"/>
-    <xacro:property name="wheel_joint_z" value="0.05"/>
+    <xacro:property name="wheel_radius" value="0.165"/>
+    <xacro:property name="wheel_length" value="0.116"/>
+    <xacro:property name="wheel_joint_x" value="0.249"/>
+    <xacro:property name="wheel_joint_y" value="0.2951"/>
+    <xacro:property name="wheel_joint_z" value="${0.2445-wheel_radius}"/>
+    <xacro:property name="gaps"  value="0.141"/>
     <xacro:property name="caster_mass"    value="0.5" />
     <xacro:property name="caster_radius"  value="0.015"/> <!-- wheel_radius - ( base_length/2 - wheel_joint_z) -->
@@ -23,4 +31,7 @@
     <material name="gray">
         <color rgba="0.75 0.75 0.75 1"/>
+    </material>
+    <material name="white">
+        <color rgba="1 0.9843 0.9412 1"/>
     </material>
     <!-- Macro for inertia matrix -->
@@ -41,8 +52,16 @@
         </inertial>
     </xacro:macro>
+    <xacro:macro name="default_inertial" params="mass">
+               <inertial>
+                       <mass value="${mass}" />
+                       <inertia ixx="1.0" ixy="0.0" ixz="0.0"
+                                iyy="1.0" iyz="0.0"
+                                izz="1.0" />
+               </inertial>
+    </xacro:macro>
     <!-- Macro for robot wheel -->
-    <xacro:macro name="wheel" params="prefix reflect">
+    <xacro:macro name="wheel" params="prefix reflect1 reflect2">
         <joint name="${prefix}_wheel_joint" type="continuous">
-            <origin xyz="0 ${reflect*wheel_joint_y} ${-wheel_joint_z}" rpy="0 0 0"/>
+            <origin xyz=" ${reflect1*wheel_joint_x} ${reflect2*wheel_joint_y} ${-wheel_joint_z}" rpy="0 0 0"/>
             <parent link="base_link"/>
             <child link="${prefix}_wheel_link"/>
@@ -55,5 +74,5 @@
                     <cylinder radius="${wheel_radius}" length = "${wheel_length}"/>
                 </geometry>
-                <material name="gray" />
+                <material name="black" />
             </visual>
             <collision>
@@ -80,32 +99,4 @@
         </transmission>
     </xacro:macro>
-    <!-- Macro for robot caster -->
-    <xacro:macro name="caster" params="prefix reflect">
-        <joint name="${prefix}_caster_joint" type="continuous">
-            <origin xyz="${reflect*caster_joint_x} 0 ${-(base_length/2 + caster_radius)}" rpy="0 0 0"/>
-            <parent link="base_link"/>
-            <child link="${prefix}_caster_link"/>
-            <axis xyz="0 1 0"/>
-        </joint>
-        <link name="${prefix}_caster_link">
-            <visual>
-                <origin xyz="0 0 0" rpy="0 0 0"/>
-                <geometry>
-                    <sphere radius="${caster_radius}" />
-                </geometry>
-                <material name="black" />
-            </visual>
-            <collision>
-                <origin xyz="0 0 0" rpy="0 0 0"/>
-                <geometry>
-                    <sphere radius="${caster_radius}" />
-                </geometry>
-            </collision>
-            <sphere_inertial_matrix  m="${caster_mass}" r="${caster_radius}" />
-        </link>
-        <gazebo reference="${prefix}_caster_link">
-            <material>Gazebo/Black</material>
-        </gazebo>
-    </xacro:macro>
     <xacro:macro name="mbot_base_gazebo">
         <link name="base_footprint">
@@ -121,5 +112,5 @@
         </gazebo>
         <joint name="base_footprint_joint" type="fixed">
-            <origin xyz="0 0 ${base_length/2 + caster_radius*2}" rpy="0 0 0" />
+            <origin xyz="0 0 ${base_length/2 + gaps}" rpy="0 0 0" />
             <parent link="base_footprint"/>
             <child link="base_link" />
@@ -129,27 +120,49 @@
                 <origin xyz=" 0 0 0" rpy="0 0 0" />
                 <geometry>
-                    <cylinder length="${base_length}" radius="${base_radius}"/>
+                    <box size="${base_x} ${base_y} ${base_z}" />
                 </geometry>
-                <material name="yellow" />
+                <material name="white" />
             </visual>
             <collision>
                 <origin xyz=" 0 0 0" rpy="0 0 0" />
                 <geometry>
-                    <cylinder length="${base_length}" radius="${base_radius}"/>
+                    <box size="${base_x} ${base_y} ${base_z}" />
                 </geometry>
             </collision>
-            <cylinder_inertial_matrix  m="${base_mass}" r="${base_radius}" h="${base_length}" />
+            <xacro:default_inertial mass="10"/>
         </link>
         <gazebo reference="base_link">
             <material>Gazebo/Blue</material>
         </gazebo>
-        <wheel prefix="left"  reflect="-1"/>
-        <wheel prefix="right" reflect="1"/>
-        <caster prefix="front" reflect="-1"/>
-        <caster prefix="back"  reflect="1"/>
-        <!-- controller -->
+        <link name="base_box">
+            <visual>
+                <origin xyz=" 0 0 0" rpy="0 0 0" />
+                <geometry>
+                    <box size="${base_box_x} ${base_box_y} ${base_box_z}" />
+                </geometry>
+                <material name="white" />
+            </visual>
+            <collision>
+                <origin xyz=" 0 0 0" rpy="0 0 0" />
+                <geometry>
+                    <box size="${base_box_x} ${base_box_y} ${base_box_z}" />
+                </geometry>
+            </collision>
+            <xacro:default_inertial mass="10"/>
+        </link>
+        <joint name="base_box_joint" type="fixed">
+            <origin xyz="0 0 ${(base_z + base_box_z)/2}" rpy="0 0 0" />
+            <parent link="base_link"/>
+            <child link="base_box" />
+        </joint>
+        <wheel prefix="right_front" reflect1="1" reflect2="-1"/>
+        <wheel prefix="right_back"  reflect1="-1" reflect2="-1"/>
+        <wheel prefix="left_front"  reflect1="1" reflect2="1"/>
+        <wheel prefix="left_back"  reflect1="-1" reflect2="1"/>
+          <!-- controller -->
+       <!-- controller -->
         <gazebo>
             <plugin name="differential_drive_controller"
-                    filename="libgazebo_ros_diff_drive.so">
+                    filename="libgazebo_ros_skid_steer_drive.so">
                 <rosDebugLevel>Debug</rosDebugLevel>
                 <publishWheelTF>true</publishWheelTF>
@@ -160,6 +173,8 @@
                 <updateRate>100.0</updateRate>
                 <legacyMode>true</legacyMode>
-                <leftJoint>left_wheel_joint</leftJoint>
-                <rightJoint>right_wheel_joint</rightJoint>
+                <leftFrontJoint>left_front_wheel_joint</leftFrontJoint>
+                <leftRearJoint>left_back_wheel_joint</leftRearJoint>
+                <rightFrontJoint>right_front_wheel_joint</rightFrontJoint>
+                <rightRearJoint>right_back_wheel_joint</rightRearJoint>
                 <wheelSeparation>${wheel_joint_y*2}</wheelSeparation>
                 <wheelDiameter>${2*wheel_radius}</wheelDiameter>
