Commit message: add some nav docs

File: NavigationPlanning/dlonng_ws/src/agilex_description/urdf/xacro/gazebo/agilex_mini_gazebo.xacro (robot description, xacro)
@@ -1,5 +1,4 @@
 <?xml version="1.0"?>
-<robot name="agilex_mini"
-    xmlns:xacro="http://www.ros.org/wiki/xacro">
+<robot name="agilex_mini" xmlns:xacro="http://www.ros.org/wiki/xacro">
     <xacro:property name="length_wheel" value="0.045" />
     <xacro:property name="radius_wheel" value="0.070" />
@@ -12,4 +11,10 @@
     <xacro:property name="width_sensor_support" value="0.23" />
     <xacro:property name="height_sensor_support" value="0.23" />
+    <xacro:property name="imu_length_x" value="0.06" />
+    <xacro:property name="imu_length_y" value="0.04" />
+    <xacro:property name="imu_length_z" value="0.022" />
+    <xacro:property name="imu_offset_x" value="0" />
+    <xacro:property name="imu_offset_y" value="0" />
+    <xacro:property name="imu_offset_z" value="${imu_length_z/2 + height_body}" />
     <xacro:macro name="default_inertial" params="mass">
         <inertial>
@@ -146,4 +151,27 @@
         <origin rpy="-1.5707 0 0" xyz="-${0.5 * width_body - radius_wheel} -${0.5 * length_body + 0.8 * length_wheel} 0"/>
     </joint>
+    <link name="imu_link">
+        <visual>
+            <origin xyz=" 0 0 0" rpy="0 0 0" />
+            <geometry>
+                <box size="${imu_length_x} ${imu_length_y} ${imu_length_z}" />
+            </geometry>
+            <material name="yellow">
+                <color rgba="1 0.4 0 1"/>
+            </material>
+        </visual>
+        <collision>
+            <origin xyz=" 0 0 0" rpy="0 0 0" />
+            <geometry>
+                <box size="${imu_length_x} ${imu_length_y} ${imu_length_z}" />
+            </geometry>
+        </collision>
+        <xacro:default_inertial mass="10"/>
+    </link>
+    <joint name="imu_joint" type="fixed">
+        <origin xyz="${imu_offset_x} ${imu_offset_y} ${imu_offset_z}" rpy="0 0 0" />
+        <parent link="base_link"/>
+        <child link="imu_link"/>
+    </joint>
     <link name="sensor_support">
         <visual>

Commit message: add nav lab1 lab2 lab3

File: NavigationPlanning/dlonng_ws/src/agilex_description/urdf/xacro/gazebo/agilex_mini_gazebo.xacro (robot description, xacro)
@@ -23,23 +23,5 @@
         </inertial>
     </xacro:macro>
-    <link name="base_footprint">
-        <visual>
-            <geometry>
-                <box size="0.001 0.001 0.001"/>
-            </geometry>
-            <origin rpy="0 0 0" xyz="0 0 0"/>
-        </visual>
-        <xacro:default_inertial mass="0.0001"/>
-    </link>
-    <gazebo reference="base_footprint">
-        <material>Gazebo/Green</material>
-        <turnGravityOff>false</turnGravityOff>
-    </gazebo>
     <xacro:include filename="$(find agilex_description)/urdf/xacro/gazebo/agilex_mini_gazebo.gazebo" />
-    <joint name="base_footprint_joint" type="fixed">
-        <origin xyz="0 0 0" />
-        <parent link="base_footprint" />
-        <child link="base_link" />
-    </joint>
     <link name="base_link">
         <visual>
